File: eagle/openmv3/shields/lcd/lcd.brd (EAGLE design)
At the start: 37.8 x 47.5 mm, 12 parts, among them J1 1X8, J2 1X8, Q1 MOSFET

Commit message: Update design files
Parts:
- C2: value 10uF -> 4.7uF; device sfe:0805 -> sfe:0603-CAP
- R3: value 10k -> 2.2K
- moved R3 0.40 mm to (12.2, 4.83)
- moved SJ1 0.38 mm to (9.27, 4.45)
- moved R4 0.28 mm to (15.7, 7.75)
- moved R6 0.28 mm to (14.0, 4.83)
- moved Q1 0.18 mm to (16.6, 4.83)
- moved C2 0.13 mm to (25.5, 4.83)
- moved R2 0.13 mm to (21.8, 4.83)
Routing:
- net LED: track 3.42 -> 2.61 mm
- net RST: track 19.2 -> 18.6 mm
