File: eagle/openmv3/shields/lcd/lcd.sch (EAGLE design)
At the start: 12 parts, among them J1 1X8, J2 1X8, Q1 MOSFET

Commit message: Update design files
Parts:
- C2: value 10uF -> 4.7uF; device sfe:CAP0805 -> sfe:CAP0603-CAP
- R3: value 10k -> 2.2K
Other:
- moved on the sheet: FB1, Q1, R3, R4, R6
